Commit message: Zmienia nazwę paczki opisu robota, usuwa niepotrzebne pliki

File: src/slambot_description/urdf/mapping_robot_v1.xacro (robot description, xacro)
@@ -1,7 +1,7 @@
 <?xml version="1.0" ?>
-<robot name="mapping_robot_v1" xmlns:xacro="http://www.ros.org/wiki/xacro">
-<xacro:include filename="$(find mapping_robot_v1_description)/urdf/materials.xacro" />
-<xacro:include filename="$(find mapping_robot_v1_description)/urdf/mapping_robot_v1.trans" />
-<xacro:include filename="$(find mapping_robot_v1_description)/urdf/mapping_robot_v1.gazebo" />
+<robot name="slambot" xmlns:xacro="http://www.ros.org/wiki/xacro">
+<xacro:include filename="$(find slambot_description)/urdf/materials.xacro" />
+<xacro:include filename="$(find slambot_description)/urdf/mapping_robot_v1.trans" />
+<xacro:include filename="$(find slambot_description)/urdf/mapping_robot_v1.gazebo" />
 <link name="base_link">
   <inertial>
@@ -13,5 +13,5 @@
     <origin xyz="0 0 0" rpy="0 0 0"/>
     <geometry>
-      <mesh filename="package://mapping_robot_v1_description/meshes/base_link.stl" scale="0.001 0.001 0.001"/>
+      <mesh filename="package://slambot_description/meshes/base_link.stl" scale="0.001 0.001 0.001"/>
     </geometry>
     <material name="silver"/>
@@ -20,5 +20,5 @@
     <origin xyz="0 0 0" rpy="0 0 0"/>
     <geometry>
-      <mesh filename="package://mapping_robot_v1_description/meshes/base_link.stl" scale="0.001 0.001 0.001"/>
+      <mesh filename="package://slambot_description/meshes/base_link.stl" scale="0.001 0.001 0.001"/>
     </geometry>
   </collision>
@@ -33,5 +33,5 @@
     <origin xyz="-0.1 -0.084 0.007" rpy="0 0 0"/>
     <geometry>
-      <mesh filename="package://mapping_robot_v1_description/meshes/front_left_link_1.stl" scale="0.001 0.001 0.001"/>
+      <mesh filename="package://slambot_description/meshes/front_left_link_1.stl" scale="0.001 0.001 0.001"/>
     </geometry>
     <material name="silver"/>
@@ -40,5 +40,5 @@
     <origin xyz="-0.1 -0.084 0.007" rpy="0 0 0"/>
     <geometry>
-      <mesh filename="package://mapping_robot_v1_description/meshes/front_left_link_1.stl" scale="0.001 0.001 0.001"/>
+      <mesh filename="package://slambot_description/meshes/front_left_link_1.stl" scale="0.001 0.001 0.001"/>
     </geometry>
   </collision>
@@ -53,5 +53,5 @@
     <origin xyz="0.1 -0.084 0.007" rpy="0 0 0"/>
     <geometry>
-      <mesh filename="package://mapping_robot_v1_description/meshes/back_left_link_1.stl" scale="0.001 0.001 0.001"/>
+      <mesh filename="package://slambot_description/meshes/back_left_link_1.stl" scale="0.001 0.001 0.001"/>
     </geometry>
     <material name="silver"/>
@@ -60,5 +60,5 @@
     <origin xyz="0.1 -0.084 0.007" rpy="0 0 0"/>
     <geometry>
-      <mesh filename="package://mapping_robot_v1_description/meshes/back_left_link_1.stl" scale="0.001 0.001 0.001"/>
+      <mesh filename="package://slambot_description/meshes/back_left_link_1.stl" scale="0.001 0.001 0.001"/>
     </geometry>
   </collision>
@@ -75,5 +75,5 @@
     <origin xyz="0.1 0.084 0.007" rpy="0 0 0"/>
     <geometry>
-      <mesh filename="package://mapping_robot_v1_description/meshes/back_right_link_1.stl" scale="0.001 0.001 0.001"/>
+      <mesh filename="package://slambot_description/meshes/back_right_link_1.stl" scale="0.001 0.001 0.001"/>
     </geometry>
     <material name="silver"/>
@@ -82,5 +82,5 @@
     <origin xyz="0.1 0.084 0.007" rpy="0 0 0"/>
     <geometry>
-      <mesh filename="package://mapping_robot_v1_description/meshes/back_right_link_1.stl" scale="0.001 0.001 0.001"/>
+      <mesh filename="package://slambot_description/meshes/back_right_link_1.stl" scale="0.001 0.001 0.001"/>
     </geometry>
   </collision>
@@ -95,5 +95,5 @@
     <origin xyz="-0.1 0.084 0.007" rpy="0 0 0"/>
     <geometry>
-      <mesh filename="package://mapping_robot_v1_description/meshes/front_right_link_1.stl" scale="0.001 0.001 0.001"/>
+      <mesh filename="package://slambot_description/meshes/front_right_link_1.stl" scale="0.001 0.001 0.001"/>
     </geometry>
     <material name="silver"/>
@@ -102,5 +102,5 @@
     <origin xyz="-0.1 0.084 0.007" rpy="0 0 0"/>
     <geometry>
-      <mesh filename="package://mapping_robot_v1_description/meshes/front_right_link_1.stl" scale="0.001 0.001 0.001"/>
+      <mesh filename="package://slambot_description/meshes/front_right_link_1.stl" scale="0.001 0.001 0.001"/>
     </geometry>
   </collision>

File: src/slambot_description/urdf/materials.xacro (robot description, xacro)
@@ -1,4 +1,4 @@
 <?xml version="1.0" ?>
-<robot name="mapping_robot_v1" xmlns:xacro="http://www.ros.org/wiki/xacro" >
+<robot name="slambot" xmlns:xacro="http://www.ros.org/wiki/xacro" >
 <material name="silver">
   <color rgba="0.700 0.700 0.700 1.000"/>
